Commit message: some fix

File: src/robot_descriptor/descriptor/camera_frames.xacro (robot description, xacro)
@@ -2,5 +2,5 @@
 <robot xmlns:xacro="http://www.ros.org/wiki/xacro">
   <joint name="camera_depth_optical_joint" type="fixed">
-    <parent link="camera_depth_link"/>
+    <parent link="camera_link"/>
     <child link="camera_depth_optical_frame"/>
     <origin xyz="0.02 0.02 0.035"
@@ -15,5 +15,5 @@
   </joint>
   <link name="camera_color_optical_frame"/>
-  <gazebo reference="camera_depth_link">
+  <gazebo reference="camera_link">
     <preserveFixedJoint>true</preserveFixedJoint>
     <self_collide>false</self_collide>

File: src/robot_descriptor/descriptor/depth_camera.xacro (robot description, xacro)
@@ -2,10 +2,10 @@
 <robot xmlns:xacro="http://www.ros.org/wiki/xacro">
     <!-- DEPTH CAMERA -->
-    <joint name="camera_depth_joint" type="fixed">
+    <joint name="camera_joint" type="fixed">
         <parent link="chassis"/>
-        <child link="camera_depth_link"/>
+        <child link="camera_link"/>
         <origin xyz="0.140 0 0.12" rpy="0 0 0"/>
     </joint>
-    <link name="camera_depth_link">
+    <link name="camera_link">
         <visual>
             <origin xyz="0.0 0 0.0" rpy="${pi} ${2*pi} ${pi/2}"/>
