Commit message: 8 May PC changes

File: src/robot_descriptor/descriptor/camera.xacro (robot description, xacro)
@@ -5,9 +5,9 @@
         <parent link="chassis"/>
         <child link="camera_rgb_link"/>
-        <origin xyz="0.135 -0.03 0.040" rpy="0 0 0"/>
+        <origin xyz="0.140 -0.03 0.040" rpy="0 0 0"/>
     </joint>
     <link name="camera_rgb_link">
         <visual>
-            <origin xyz="-0.138 0.032 -0.04"
+            <origin xyz="-0.144 0.032 -0.04"
                     rpy="${-pi/2} ${-pi} ${-pi/2}"/>
             <geometry>
@@ -18,4 +18,5 @@
         </visual>
     </link>
+    <!-- Optical frame (ROS camera convention) -->
     <joint name="camera_rgb_optical_joint" type="fixed">
         <parent link="camera_rgb_link"/>
@@ -25,36 +26,40 @@
     </joint>
     <link name="camera_rgb_optical_link"/>
+    <!-- Gazebo camera sensor -->
     <gazebo reference="camera_rgb_link">
-    <self_collide>false</self_collide>
-    <material>Gazebo/Green</material>
-    <preserveFixedJoint>true</preserveFixedJoint>
-    <sensor name="modul3_wide" type="camera">
-        <pose>0 0 0 0 0 0</pose>
-        <always_on>true</always_on>
-        <update_rate>10</update_rate>
-        <visualize>true</visualize>
-        <camera>
-       <camera_info_topic>/camera/rgb/camera_info</camera_info_topic>
-        <horizontal_fov>1.78</horizontal_fov>
-        <image>
-            <width>640</width>
-            <height>480</height>
-            <format>R8G8B8</format>
-        </image>
-        <clip>
-        <near>0.5</near>
-        <far>3.0</far>
-        </clip>
-        <distortion>
-            <k1>-0.02</k1>
-            <k2>0.01</k2>
-            <k3>0.0</k3>
-            <p1>0.0</p1>
-            <p2>0.0</p2>
-        </distortion>
-        </camera>
-        <topic>camera/rgb/image_raw</topic>
-        <gz_frame_id>camera_rgb_optical_link</gz_frame_id>
-    </sensor>
+        <self_collide>false</self_collide>
+        <material>Gazebo/Green</material>
+        <preserveFixedJoint>true</preserveFixedJoint>
+        <sensor name="modul3_wide" type="camera">
+            <pose>0 0 0 0 0 0</pose>
+            <always_on>true</always_on>
+            <update_rate>30</update_rate>
+            <visualize>true</visualize>
+            <camera>
+                <camera_info_topic>/camera/rgb/camera_info</camera_info_topic>
+                <horizontal_fov>1.78</horizontal_fov>
+                <image>
+                    <width>640</width>
+                    <height>480</height>
+                    <format>R8G8B8</format>
+                </image>
+                <clip>
+                    <near>0.05</near>
+                    <far>8.0</far>
+                </clip>
+                <distortion>
+                    <k1>-0.02</k1>
+                    <k2>0.01</k2>
+                    <k3>0.0</k3>
+                    <p1>0.0</p1>
+                    <p2>0.0</p2>
+                </distortion>
+                <!-- CHANGED: aggiunto optical_frame_id -->
+                <optical_frame_id>camera_rgb_optical_link</optical_frame_id>
+            </camera>
+            <topic>camera/rgb/image_raw</topic>
+            <!-- REMOVED: questa riga rompeva l'orientazione -->
+            <!-- <gz_frame_id>camera_rgb_optical_link</gz_frame_id> -->
+        </sensor>
     </gazebo>
 </robot>

File: src/robot_descriptor/descriptor/camera_frames.xacro (robot description, xacro)
@@ -1,4 +1,5 @@
 <?xml version="1.0"?>
 <robot xmlns:xacro="http://www.ros.org/wiki/xacro">
+  <!-- Depth optical frame -->
   <joint name="camera_depth_optical_joint" type="fixed">
     <parent link="camera_link"/>
@@ -8,4 +9,5 @@
   </joint>
   <link name="camera_depth_optical_frame"/>
+  <!-- Color optical frame -->
   <joint name="camera_color_optical_joint" type="fixed">
     <parent link="camera_depth_optical_frame"/>
@@ -15,12 +17,15 @@
   </joint>
   <link name="camera_color_optical_frame"/>
+  <!-- Gazebo RGBD camera sensor -->
   <gazebo reference="camera_link">
     <preserveFixedJoint>true</preserveFixedJoint>
     <self_collide>false</self_collide>
-    <sensor name="d435i_depth" type="rgbd_camera">
+    <sensor name="d435i_rgbd" type="rgbd_camera">
       <pose>0 0 0 0 0 0</pose>
       <always_on>true</always_on>
       <update_rate>10</update_rate>
-      <visualize>true</visualize> <topic>camera/rgbd</topic> <camera>
+      <visualize>true</visualize>
+      <topic>camera/rgbd</topic>
+      <camera>
         <horizontal_fov>1.518</horizontal_fov>
         <image>
@@ -31,9 +36,9 @@
         <clip>
           <near>0.1</near>
-          <far>8.0</far>
+          <far>12.0</far>
         </clip>
-        <optical_frame_id>camera_depth_optical_frame</optical_frame_id>
+        <!-- ROS optical frame -->
+        <optical_frame_id>camera_link</optical_frame_id>
       </camera>
-      <gz_frame_id>camera_depth_link</gz_frame_id>
       <camera_info_topic>camera/rgbd/camera_info</camera_info_topic>
       <depth_topic>camera/rgbd/depth_image</depth_topic>

File: src/robot_descriptor/descriptor/lidar.xacro (robot description, xacro)
@@ -27,5 +27,5 @@
         <visualize>false</visualize>
         <topic>scan</topic>
-        <ignition_frame_id>laser_frame</ignition_frame_id>
+        <gz_frame_id>laser_frame</gz_frame_id>
         <lidar>
         <scan>

File: src/robot_descriptor/descriptor/robot_core.xacro (robot description, xacro)
@@ -38,5 +38,5 @@
   </material>
   <material name="green">
-    <color rgba="0 0.8 0 0.95"/>
+    <color rgba="0 0.8 0 1"/>
   </material>
   <material name="grey">
@@ -104,5 +104,5 @@
     <visualize>true</visualize>
     <topic>imu</topic>
-    <ignition_frame_id>imu</ignition_frame_id>
+    <gz_frame_id>imu</gz_frame_id>
     <plugin filename="libignition-gazebo-imu-system.so" name="ignition::gazebo::systems::Imu">
     </plugin>
