Commit message: new urdf

File: src/robot_descriptor/descriptor/depth_camera.xacro (robot description, xacro)
@@ -5,11 +5,11 @@
         <parent link="chassis"/>
         <child link="camera_link"/>
-        <origin xyz="0.140 0 0.12" rpy="0 0 0"/>
+        <origin xyz="0.11 0.0105 0.1285" rpy="0 0 0"/>
     </joint>
     <link name="camera_link">
         <visual>
-            <origin xyz="0.0 0 0.0" rpy="${pi} ${2*pi} ${pi/2}"/>
+            <origin xyz="0.0 -0.013 0.0" rpy="${pi/2} ${0} ${pi/2}"/>
             <geometry>
-                <mesh filename="package://robot_descriptor/meshes/d435i.stl"
+                <mesh filename="package://robot_descriptor/meshes/IntelRealsense_D435i.stl"
                       scale="0.001 0.001 0.001"/>
            </geometry>

File: src/robot_descriptor/descriptor/lidar.xacro (robot description, xacro)
@@ -4,9 +4,9 @@
         <parent link="base_link"/>
         <child link="laser_frame"/>
-        <origin xyz="-0.025 0 ${wheel_radius+0.187}" rpy="0 3.14159265359 1.57079"/>
+        <origin xyz="0.075 0 ${wheel_radius+0.181}" rpy="0 3.14159265359 1.57079"/>
     </joint>
     <link name="laser_frame">
         <visual>
-            <origin xyz="0.0025 0 0.045" rpy=" -1.57079  0   3.14159265359"/>
+            <origin xyz="0.0035 -0.0 0.041" rpy=" -1.57079  0   3.14159265359"/>
             <geometry>
                 <mesh filename="package://robot_descriptor/meshes/lidar.stl" scale="0.001 0.001 0.001"/>

File: src/robot_descriptor/descriptor/robot.urdf.xacro (robot description, xacro)
@@ -5,8 +5,8 @@
     <xacro:include filename="robot_core.xacro" />
     <xacro:include filename="lidar.xacro" />
-    <xacro:include filename="camera.xacro" />
+      <!-- <xacro:include filename="camera.xacro" /> -->
     <xacro:include filename="depth_camera.xacro" />
     <xacro:if value="$(arg use_sim_camera)">
-        <xacro:include filename="camera_frames.xacro"/>
+        <!--<xacro:include filename="camera_frames.xacro"/>-->
     </xacro:if>
 </robot>

File: src/robot_descriptor/descriptor/robot_core.xacro (robot description, xacro)
@@ -26,11 +26,11 @@
   </material>
   <material name="blue">
-    <color rgba="0.2 0.2 1 0.9"/>
+    <color rgba="0.2 0.2 1 1"/>
   </material>
   <material name="black">
-    <color rgba="0 0 0 0.9"/>
+    <color rgba="0 0 0 0.99"/>
   </material>
  <material name="light_black">
-    <color rgba="0.1 0.1 0.1 0.999"/>
+    <color rgba="0.1 0.1 0.1 1"/>
   </material>
   <material name="red">
@@ -41,5 +41,5 @@
   </material>
   <material name="grey">
-    <color rgba="0.647 0.647 0.647 0.95"/>
+    <color rgba="0.647 0.647 0.647 1"/>
   </material>
   <!-- ================= BASE LINK ================= -->
@@ -62,5 +62,5 @@
       <origin xyz="0 0.0035 0" rpy="1.5708 0 1.5708"/>
       <geometry>
-        <mesh filename="package://robot_descriptor/meshes/chassis.stl"
+        <mesh filename="package://robot_descriptor/meshes/chassis_main.stl"
               scale="0.001 0.001 0.001"/>
       </geometry>
