Commit message: change lidar port and lidar frame name

File: src/robot_descriptor/descriptor/lidar.xacro (robot description, xacro)
@@ -3,8 +3,8 @@
     <joint name="laser_joint" type="fixed">
         <parent link="base_link"/>
-        <child link="laser_frame"/>
+        <child link="laser_link"/>
         <origin xyz="0.075 0 ${wheel_radius+0.181}" rpy="0 3.14159265359 1.57079"/>
     </joint>
-    <link name="laser_frame">
+    <link name="laser_link">
         <visual>
             <origin xyz="0.0035 -0.0 0.041" rpy=" -1.57079  0   3.14159265359"/>
@@ -18,5 +18,5 @@
         </xacro:inertial_cylinder>
     </link>
-    <gazebo reference="laser_frame">
+    <gazebo reference="laser_link">
     <material>Gazebo/Black</material>
     <self_collide>false</self_collide>
@@ -27,5 +27,5 @@
         <visualize>false</visualize>
         <topic>scan</topic>
-        <gz_frame_id>laser_frame</gz_frame_id>
+        <gz_frame_id>laser_link</gz_frame_id>
         <lidar>
         <scan>
